File: design/atboard.kicad_pcb (KiCad board)
At the start: 2 copper layers, 36.8 x 53.3 mm, 8 parts, among them J1 AVR_SPI, J2 RIGHT_CONNECTOR, J3 LEFT_CONNECTOR, J4 POWER, U1 ATmega328-PU, Y1 8 MHz

Commit message: everything is wired up. saving before adding a ground plane
Routing:
- net /MOSI: track 36.4 -> 40.2 mm
- net /28: track 0.00 -> 3.81 mm
- net /27: track 0.00 -> 3.81 mm
- net /26: track 0.00 -> 3.81 mm
- net /25: track 0.00 -> 3.81 mm
- net /24: track 0.00 -> 3.81 mm
- net /23: track 0.00 -> 3.81 mm
- net /21: track 0.00 -> 3.81 mm
- net /20: track 0.00 -> 3.81 mm
- net /16: track 0.00 -> 3.81 mm
- net /15: track 0.00 -> 3.81 mm
Changed lines of the file:
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@@
     (thickness 1.6)
     (drawings 4)
-    (tracks 60)
+    (tracks 71)
     (zones 0)
     (modules 8)
@@
   (segment (start 88.9 54.61) (end 86.36 57.15) (width 0.25) (layer F.Cu) (net 17))
   (segment (start 88.9 50.8) (end 88.9 54.61) (width 0.25) (layer F.Cu) (net 17))
+  (segment (start 88.9 85.09) (end 92.71 85.09) (width 0.25) (layer F.Cu) (net 17))
+  (segment (start 88.9 90.17) (end 92.71 90.17) (width 0.25) (layer F.Cu) (net 18))
+  (segment (start 88.9 87.63) (end 92.71 87.63) (width 0.25) (layer F.Cu) (net 19))
+  (segment (start 88.9 77.47) (end 92.71 77.47) (width 0.25) (layer F.Cu) (net 20))
+  (segment (start 88.9 74.93) (end 92.71 74.93) (width 0.25) (layer F.Cu) (net 21))
+  (segment (start 88.9 69.85) (end 92.71 69.85) (width 0.25) (layer F.Cu) (net 22))
+  (segment (start 88.9 67.31) (end 92.71 67.31) (width 0.25) (layer F.Cu) (net 23))
+  (segment (start 88.9 64.77) (end 92.71 64.77) (width 0.25) (layer F.Cu) (net 24))
+  (segment (start 88.9 62.23) (end 92.71 62.23) (width 0.25) (layer F.Cu) (net 25))
+  (segment (start 88.9 59.69) (end 92.71 59.69) (width 0.25) (layer F.Cu) (net 26))
+  (segment (start 88.9 57.15) (end 92.71 57.15) (width 0.25) (layer F.Cu) (net 27))
   (segment (start 81.28 90.17) (end 76.2 90.17) (width 0.25) (layer F.Cu) (net 28))
 )

Commit message: save work
Routing:
- added copper zone on F.Cu, net GND
Changed lines of the file:
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@@
   (segment (start 88.9 57.15) (end 92.71 57.15) (width 0.25) (layer F.Cu) (net 27))
   (segment (start 81.28 90.17) (end 76.2 90.17) (width 0.25) (layer F.Cu) (net 28))
+  (zone (net 1) (net_name GND) (layer F.Cu) (hatch edge 0.508)
+    (connect_pads (clearance 0.508))
+    (min_thickness 0.254)
+    (fill yes (arc_segments 32) (thermal_gap 0.508) (thermal_bridge_width 0.508))
+    (polygon
+      (pts
+        (xy 64.77 43.18) (xy 99.06 43.18) (xy 99.06 93.98) (xy 64.77 93.98)
+      )
+    )
+  )
 )
