File: design/atmega-dip/_autosave-atmega-dip.kicad_pcb (KiCad board)
At the start: 2 copper layers, 29.2 x 63.5 mm, 8 parts, among them J1 AVR_SPI, J2 RIGHT_CONNECTOR, J3 LEFT_CONNECTOR, J4 POWER, U1 ATmega328-PU, Y1 8 MHz

Commit message: finish the routing
Routing:
- net /RST: track 5.16 -> 43.2 mm, vias 0 -> 1
Changed lines of the file:
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@@
     (thickness 1.6)
     (drawings 10)
-    (tracks 67)
+    (tracks 74)
     (zones 0)
     (modules 8)
@@
     (descr "Crystal THT HC-49-4H http://5hertz.com/pdfs/04404_D.pdf")
     (tags "THT crystalHC-49-4H")
-    (fp_text reference Y1 (at 6.858 3.556 180) (layer F.SilkS)
+    (fp_text reference Y1 (at 6.858 3.81 180) (layer F.SilkS)
       (effects (font (size 1 1) (thickness 0.15)))
     )
@@
   (segment (start 144.861399 57.068601) (end 146.05 55.88) (width 0.25) (layer F.Cu) (net 7))
   (segment (start 145.542 103.378) (end 144.018 103.378) (width 0.25) (layer F.Cu) (net 7))
-  (segment (start 136.144 54.356) (end 136.084999 54.415001) (width 0.25) (layer F.Cu) (net 8))
   (segment (start 134.874 75.438) (end 132.842 75.438) (width 0.25) (layer F.Cu) (net 8))
   (segment (start 135.128 75.438) (end 134.874 75.438) (width 0.25) (layer F.Cu) (net 8))
   (segment (start 137.922 75.438) (end 135.128 75.438) (width 0.25) (layer F.Cu) (net 8))
+  (segment (start 148.59 58.42) (end 154.686 58.42) (width 0.25) (layer F.Cu) (net 8))
+  (segment (start 154.686 58.42) (end 154.686 71.374) (width 0.25) (layer F.Cu) (net 8))
+  (segment (start 154.686 71.374) (end 153.924 72.136) (width 0.25) (layer F.Cu) (net 8))
+  (via (at 146.558 72.136) (size 0.8) (drill 0.4) (layers F.Cu B.Cu) (net 8))
+  (segment (start 153.924 72.136) (end 146.558 72.136) (width 0.25) (layer F.Cu) (net 8))
+  (segment (start 137.922 74.388) (end 137.922 75.438) (width 0.25) (layer B.Cu) (net 8))
+  (segment (start 140.174 72.136) (end 137.922 74.388) (width 0.25) (layer B.Cu) (net 8))
+  (segment (start 146.558 72.136) (end 140.174 72.136) (width 0.25) (layer B.Cu) (net 8))
   (segment (start 145.542 108.458) (end 150.622 108.458) (width 0.25) (layer F.Cu) (net 9))
   (segment (start 145.542 105.918) (end 150.622 105.918) (width 0.25) (layer F.Cu) (net 10))
