File: design/atmega-dip/atmega-dip.kicad_pcb (KiCad board)
At the start: 2 copper layers, 29.2 x 50.8 mm, 8 parts, among them J1 AVR_SPI, J2 RIGHT_CONNECTOR, J3 LEFT_CONNECTOR, J4 POWER, U1 ATmega328-PU, Y1 8 MHz

Commit message: still having routing to do
Parts:
- moved C1 90.6 mm to (147.0, 65.4)
- moved C2 90.6 mm to (147.0, 69.0)
- moved Y1 72.6 mm to (137.2, 68.6), turned to 180 degrees
- moved J1 12.8 mm to (143.5, 58.4)
- moved J4 8.20 mm to (133.1, 59.4), turned to 180 degrees
- moved U1 2.09 mm to (137.9, 75.4)
- moved J2 2.09 mm to (150.6, 75.4)
- moved J3 2.09 mm to (132.8, 75.4)
Routing:
- net /MOSI: track 0.00 -> 58.0 mm
- net /MISO: track 0.00 -> 49.1 mm
- net /SCK: track 0.00 -> 47.3 mm
- net +3V3: track 0.00 -> 39.0 mm
- net /10: track 0.00 -> 37.4 mm
- net /9: track 0.00 -> 34.6 mm
- net /28: track 0.00 -> 5.08 mm
- net /27: track 0.00 -> 5.08 mm
- net /26: track 0.00 -> 5.08 mm
- net /25: track 0.00 -> 5.08 mm
- net /24: track 0.00 -> 5.08 mm
- net /23: track 0.00 -> 5.08 mm
- net /21: track 0.00 -> 5.08 mm
- net /20: track 0.00 -> 5.08 mm
- net /16: track 0.00 -> 5.08 mm
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- added copper zone on F.Cu, net GND
Other:
- board size 29.2 x 50.8 mm -> 29.2 x 63.5 mm
- board text added: "1"
- board text added: "v1.0"

Commit message: some more rerouting
Parts:
- moved C1 5.87 mm to (148.3, 71.1), turned to 90 degrees
- moved C2 5.64 mm to (148.3, 63.5), turned to 270 degrees
Routing:
- net /RST: track 5.08 -> 49.7 mm
Changed lines of the file:
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@@
-(kicad_pcb (version 20171130) (host pcbnew "(5.1.0)-1")
+(kicad_pcb (version 20171130) (host pcbnew "(5.1.0-0)")
   (general
     (thickness 1.6)
     (drawings 10)
-    (tracks 57)
+    (tracks 66)
     (zones 0)
     (modules 8)
@@
   )
   (module Capacitor_THT:C_Disc_D3.0mm_W2.0mm_P2.50mm (layer F.Cu)
-    (at 146.955001 65.415001)
+    (at 148.336 71.12 90)
     (descr "C, Disc series, Radial, pin pitch=2.50mm, , diameter*width=3*2mm^2, Capacitor")
     (tags "C Disc series Radial pin pitch 2.50mm  diameter 3mm width 2mm Capacitor")
-    (fp_text reference C1 (at 5.190999 0.116999) (layer F.SilkS)
-      (effects (font (size 1 1) (thickness 0.15)))
-    )
-    (fp_text value "22 pF" (at 1.25 2.25) (layer F.Fab)
-      (effects (font (size 1 1) (thickness 0.15)))
-    )
-    (fp_text user %R (at 1.25 0) (layer F.Fab)
+    (fp_text reference C1 (at 2.794 2.54 180) (layer F.SilkS)
+      (effects (font (size 1 1) (thickness 0.15)))
+    )
+    (fp_text value "22 pF" (at 1.016 3.81 180) (layer F.Fab) hide
+      (effects (font (size 1 1) (thickness 0.15)))
+    )
+    (fp_text user %R (at 1.25 0 180) (layer F.Fab)
       (effects (font (size 0.6 0.6) (thickness 0.09)))
     )
@@
     (fp_line (start -0.25 1) (end 2.75 1) (layer F.Fab) (width 0.1))
     (fp_line (start -0.25 -1) (end -0.25 1) (layer F.Fab) (width 0.1))
-    (pad 2 thru_hole circle (at 2.5 0) (size 1.6 1.6) (drill 0.8) (layers *.Cu *.Mask)
-      (net 1 GND))
-    (pad 1 thru_hole circle (at 0 0) (size 1.6 1.6) (drill 0.8) (layers *.Cu *.Mask)
+    (pad 2 thru_hole circle (at 2.5 0 90) (size 1.6 1.6) (drill 0.8) (layers *.Cu *.Mask)
+      (net 1 GND))
+    (pad 1 thru_hole circle (at 0 0 90) (size 1.6 1.6) (drill 0.8) (layers *.Cu *.Mask)
       (net 2 /10))
     (model ${KISYS3DMOD}/Capacitor_THT.3dshapes/C_Disc_D3.0mm_W2.0mm_P2.50mm.wrl
@@
   )
   (module Capacitor_THT:C_Disc_D3.0mm_W2.0mm_P2.50mm (layer F.Cu)
-    (at 146.955001 68.965001)
+    (at 148.336 63.5 270)
     (descr "C, Disc series, Radial, pin pitch=2.50mm, , diameter*width=3*2mm^2, Capacitor")
     (tags "C Disc series Radial pin pitch 2.50mm  diameter 3mm width 2mm Capacitor")
-    (fp_text reference C2 (at 4.936999 -0.131001) (layer F.SilkS)
-      (effects (font (size 1 1) (thickness 0.15)))
-    )
-    (fp_text value "22 pF" (at 1.25 2.25) (layer F.Fab)
+    (fp_text reference C2 (at -0.254 -2.54) (layer F.SilkS)
+      (effects (font (size 1 1) (thickness 0.15)))
+    )
+    (fp_text value "22 pF" (at 1.524 -3.81) (layer F.Fab) hide
       (effects (font (size 1 1) (thickness 0.15)))
     )
@@
       (effects (font (size 0.6 0.6) (thickness 0.09)))
     )
-    (pad 1 thru_hole circle (at 0 0) (size 1.6 1.6) (drill 0.8) (layers *.Cu *.Mask)
+    (pad 1 thru_hole circle (at 0 0 270) (size 1.6 1.6) (drill 0.8) (layers *.Cu *.Mask)
       (net 3 /9))
-    (pad 2 thru_hole circle (at 2.5 0) (size 1.6 1.6) (drill 0.8) (layers *.Cu *.Mask)
+    (pad 2 thru_hole circle (at 2.5 0 270) (size 1.6 1.6) (drill 0.8) (layers *.Cu *.Mask)
       (net 1 GND))
     (model ${KISYS3DMOD}/Capacitor_THT.3dshapes/C_Disc_D3.0mm_W2.0mm_P2.50mm.wrl
@@
       (effects (font (size 1 1) (thickness 0.15)))
     )
-    (fp_text value AVR_SPI (at 1.27 11.684 90) (layer F.Fab)
+    (fp_text value AVR_SPI (at -2.032 5.334 180) (layer F.Fab)
       (effects (font (size 1 1) (thickness 0.15)))
     )
@@
   (segment (start 145.542 98.298) (end 146.67337 98.298) (width 0.25) (layer F.Cu) (net 6))
   (segment (start 145.542 103.378) (end 150.622 103.378) (width 0.25) (layer F.Cu) (net 7))
-  (segment (start 144.861399 57.068601) (end 142.321399 57.068601) (width 0.25) (layer F.Cu) (net 7))
-  (segment (start 146.05 55.88) (end 144.861399 57.068601) (width 0.25) (layer F.Cu) (net 7))
-  (segment (start 144.018 103.378) (end 145.542 103.378) (width 0.25) (layer F.Cu) (net 7))
-  (segment (start 142.321399 57.068601) (end 142.321399 70.453583) (width 0.25) (layer F.Cu) (net 7))
-  (segment (start 142.321399 70.453583) (end 142.101978 70.673004) (width 0.25) (layer F.Cu) (net 7))
-  (segment (start 142.101978 70.673004) (end 142.101978 101.461978) (width 0.25) (layer F.Cu) (net 7))
-  (segment (start 142.101978 101.461978) (end 144.018 103.378) (width 0.25) (layer F.Cu) (net 7))
-  (segment (start 137.922 75.438) (end 132.842 75.438) (width 0.25) (layer F.Cu) (net 8))
+  (segment (start 142.101978 57.288022) (end 142.321399 57.068601) (width 0.25) (layer F.Cu) (net 7))
+  (segment (start 142.101978 101.461978) (end 142.101978 57.288022) (width 0.25) (layer F.Cu) (net 7))
+  (segment (start 144.018 103.378) (end 142.101978 101.461978) (width 0.25) (layer F.Cu) (net 7))
+  (segment (start 142.321399 57.068601) (end 144.861399 57.068601) (width 0.25) (layer F.Cu) (net 7))
+  (segment (start 144.861399 57.068601) (end 146.05 55.88) (width 0.25) (layer F.Cu) (net 7))
+  (segment (start 145.542 103.378) (end 144.018 103.378) (width 0.25) (layer F.Cu) (net 7))
+  (segment (start 148.59 58.42) (end 151.892 58.42) (width 0.25) (layer F.Cu) (net 8))
+  (segment (start 151.892 58.42) (end 151.892 54.356) (width 0.25) (layer F.Cu) (net 8))
+  (segment (start 151.892 54.356) (end 136.144 54.356) (width 0.25) (layer F.Cu) (net 8))
+  (segment (start 136.084999 54.415001) (end 136.084999 64.964999) (width 0.25) (layer F.Cu) (net 8))
+  (segment (start 136.144 54.356) (end 136.084999 54.415001) (width 0.25) (layer F.Cu) (net 8))
+  (segment (start 136.084999 64.964999) (end 135.128 65.921998) (width 0.25) (layer F.Cu) (net 8))
+  (segment (start 134.874 75.438) (end 132.842 75.438) (width 0.25) (layer F.Cu) (net 8))
+  (segment (start 135.128 65.921998) (end 135.128 75.184) (width 0.25) (layer F.Cu) (net 8))
+  (segment (start 135.128 75.184) (end 135.128 75.438) (width 0.25) (layer F.Cu) (net 8))
+  (segment (start 135.128 75.438) (end 134.874 75.438) (width 0.25) (layer F.Cu) (net 8))
+  (segment (start 137.922 75.438) (end 135.128 75.438) (width 0.25) (layer F.Cu) (net 8))
   (segment (start 145.542 108.458) (end 150.622 108.458) (width 0.25) (layer F.Cu) (net 9))
   (segment (start 145.542 105.918) (end 150.622 105.918) (width 0.25) (layer F.Cu) (net 10))

Commit message: finish the routing
Parts:
- moved C1 2.34 mm to (148.8, 68.8), turned to 0 degrees
- moved C2 1.85 mm to (148.8, 65.3), turned to 0 degrees
Routing:
- net /RST: track 49.7 -> 5.08 mm
- net /9: track 34.6 -> 52.5 mm, vias 0 -> 1
- net /10: track 37.4 -> 49.2 mm, vias 0 -> 1

Commit message: add bottom silkscreen
Routing:
- net /RST: track 5.08 -> 43.2 mm, vias 0 -> 1
Changed lines of the file:
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@@
   (general
     (thickness 1.6)
-    (drawings 10)
-    (tracks 66)
+    (drawings 11)
+    (tracks 74)
     (zones 0)
     (modules 8)
@@
     (descr "Crystal THT HC-49-4H http://5hertz.com/pdfs/04404_D.pdf")
     (tags "THT crystalHC-49-4H")
-    (fp_text reference Y1 (at 6.858 3.556 180) (layer F.SilkS)
+    (fp_text reference Y1 (at 6.858 3.81 180) (layer F.SilkS)
       (effects (font (size 1 1) (thickness 0.15)))
     )
@@
       (rotate (xyz 0 0 0))
     )
+  )
+  (gr_text v1.0 (at 130.302 112.268) (layer B.SilkS)
+    (effects (font (size 1.5 1.5) (thickness 0.3)) (justify mirror))
   )
   (gr_text v1.0 (at 153.162 112.776) (layer B.Cu)
@@
   (segment (start 135.128 75.438) (end 134.874 75.438) (width 0.25) (layer F.Cu) (net 8))
   (segment (start 137.922 75.438) (end 135.128 75.438) (width 0.25) (layer F.Cu) (net 8))
+  (segment (start 148.59 58.42) (end 154.686 58.42) (width 0.25) (layer F.Cu) (net 8))
+  (segment (start 154.686 58.42) (end 154.686 71.374) (width 0.25) (layer F.Cu) (net 8))
+  (segment (start 154.686 71.374) (end 153.924 72.136) (width 0.25) (layer F.Cu) (net 8))
+  (via (at 146.558 72.136) (size 0.8) (drill 0.4) (layers F.Cu B.Cu) (net 8))
+  (segment (start 153.924 72.136) (end 146.558 72.136) (width 0.25) (layer F.Cu) (net 8))
+  (segment (start 137.922 74.388) (end 137.922 75.438) (width 0.25) (layer B.Cu) (net 8))
+  (segment (start 140.174 72.136) (end 137.922 74.388) (width 0.25) (layer B.Cu) (net 8))
+  (segment (start 146.558 72.136) (end 140.174 72.136) (width 0.25) (layer B.Cu) (net 8))
   (segment (start 145.542 108.458) (end 150.622 108.458) (width 0.25) (layer F.Cu) (net 9))
   (segment (start 145.542 105.918) (end 150.622 105.918) (width 0.25) (layer F.Cu) (net 10))
